Commit message: phc_morph

File: body0.urdf (robot description, URDF)
Before this commit: robot robot, 8 links, 7 joints
Links:
- added link link8, mass 1; collision box size=0.4726313628223936 0.6491393354415362 0.6780312269737576; visual box size=0.4726313628223936 0.6491393354415362 0.6780312269737576
- added link link9, mass 1; collision box size=0.5349836662955243 0.2960782386452592 0.05724615280790868; visual box size=0.5349836662955243 0.2960782386452592 0.05724615280790868
- link link0: geometry collision box size=0.021763687096769235 0.5317776567400722 0.05579224059339816; visual box size=0.021763687096769235 0.5317776567400722 0.05579224059339816
- link link1: geometry collision box size=0.7169645731619687 0.5897490328007347 0.93217455492804; visual box size=0.7169645731619687 0.5897490328007347 0.93217455492804
- link link2: geometry collision box size=0.8874848008484255 0.76068286397045 0.02628548651597662; visual box size=0.8874848008484255 0.76068286397045 0.02628548651597662
- link link3: geometry collision box size=0.6137194757148703 0.4985272795982061 0.2469778701921831; visual box size=0.6137194757148703 0.4985272795982061 0.2469778701921831
- link link4: geometry collision box size=0.32788415855773057 0.811559243975822 0.7514422727504841; visual box size=0.32788415855773057 0.811559243975822 0.7514422727504841
- link link5: geometry collision box size=0.49132711511918015 0.41687121025263885 0.08822872108400515; visual box size=0.49132711511918015 0.41687121025263885 0.08822872108400515
- link link6: geometry collision box size=0.9671776241113103 0.8745506360223859 0.9493501668244368; visual box size=0.9671776241113103 0.8745506360223859 0.9493501668244368
- link link7: geometry collision box size=0.6783469612474521 0.5908745983860058 0.30164436643663395; visual box size=0.6783469612474521 0.5908745983860058 0.30164436643663395
Joints:
- removed joint link1_link2
- removed joint link1_link3
- removed joint link3_link4
- removed joint link3_link6
- removed joint link6_link7
- added joint link0_link2: type revolute, parent link0, child link2, origin xyz=-0.0005367207944518701 -0.14676835678983205 1.027896120296699 rpy=0 0 0, axis 0 1 0, limit lower=-3.14159 upper=3.14159 effort=0.0 velocity=0.0
- added joint link1_link7: type revolute, parent link1, child link7, origin xyz=0.0730771152682404 -0.15905088683469998 -0.21324769494748436 rpy=0 0 0, axis 0 0 1, limit lower=-3.14159 upper=3.14159 effort=0.0 velocity=0.0
- added joint link2_link3: type revolute, parent link2, child link3, origin xyz=-0.048605461908194925 -0.08756027766646118 0.02628548651597662 rpy=0 0 0, axis 0 1 0, limit lower=-3.14159 upper=3.14159 effort=0.0 velocity=0.0
- added joint link2_link4: type revolute, parent link2, child link4, origin xyz=-0.41560481164293145 0.4588654405196772 0.0005881428312348533 rpy=0 0 0, axis 1 0 0, limit lower=-3.14159 upper=3.14159 effort=0.0 velocity=0.0
- added joint link5_link6: type revolute, parent link5, child link6, origin xyz=0.2675284655500697 -0.3204391928984186 0.016595818480806726 rpy=0 0 0, axis 0 1 0, limit lower=-3.14159 upper=3.14159 effort=0.0 velocity=0.0
- added joint link5_link8: type revolute, parent link5, child link8, origin xyz=-0.1286800814874047 -0.22707185313962358 -0.058911196021970605 rpy=0 0 0, axis 1 0 0, limit lower=-3.14159 upper=3.14159 effort=0.0 velocity=0.0
- added joint link6_link9: type revolute, parent link6, child link9, origin xyz=-0.43902178771533207 -0.3395657193192987 0.9493501668244368 rpy=0 0 0, axis 0 1 0, limit lower=-3.14159 upper=3.14159 effort=0.0 velocity=0.0
- joint link0_link1: axis 0 1 0 -> 1 0 0; origin xyz=-0.07918220211854327 0.029860561072494102 1.2017151026887516 rpy=0 0 0 -> xyz=-0.0016856417233009193 -0.2658888283700361 1.0215263956335814 rpy=0 0 0
- joint link4_link5: axis 0 1 0 -> 0 0 1; origin xyz=0.6040245730095358 0.022663905815688 0.21443367903990912 rpy=0 0 0 -> xyz=-0.13446175029926455 -0.41724154528533297 0.13571274673672096 rpy=0 0 0
