Commit message: snakes

File: body.urdf (robot description, URDF)
Before this commit: robot robot, 3 links, 2 joints
Links:
- removed link BackLeg
- removed link FrontLeg
- removed link Torso
- added link link0, mass 1; collision box size=0.04859489333567546 0.4566873270888976 0.18447234060812828; visual box size=0.04859489333567546 0.4566873270888976 0.18447234060812828
- added link link1, mass 1; collision box size=0.4325252736494065 0.24573883548668718 0.4676630968049582; visual box size=0.4325252736494065 0.24573883548668718 0.4676630968049582
- added link link2, mass 1; collision box size=0.137498004971097 0.8809431657033127 0.17124178952639652; visual box size=0.137498004971097 0.8809431657033127 0.17124178952639652
- added link link3, mass 1; collision box size=0.9921424383479781 0.3759500970310249 0.4497203234630941; visual box size=0.9921424383479781 0.3759500970310249 0.4497203234630941
- added link link4, mass 1; collision box size=0.6415144297826938 0.41838932630841097 0.38653799620003326; visual box size=0.6415144297826938 0.41838932630841097 0.38653799620003326
Joints:
- removed joint Torso_BackLeg
- removed joint Torso_FrontLeg
- added joint link0_link1: type revolute, parent link0, child link1, origin xyz=-0.02429744666783773 0 1 rpy=0 0 0, axis 0 0 1, limit lower=-3.14159 upper=3.14159 effort=0.0 velocity=0.0
- added joint link1_link2: type revolute, parent link1, child link2, origin xyz=-0.4325252736494065 0 0 rpy=0 0 0, axis 0 0 1, limit lower=-3.14159 upper=3.14159 effort=0.0 velocity=0.0
- added joint link2_link3: type revolute, parent link2, child link3, origin xyz=-0.137498004971097 0 0 rpy=0 0 0, axis 0 0 1, limit lower=-3.14159 upper=3.14159 effort=0.0 velocity=0.0
- added joint link3_link4: type revolute, parent link3, child link4, origin xyz=-0.9921424383479781 0 0 rpy=0 0 0, axis 0 0 1, limit lower=-3.14159 upper=3.14159 effort=0.0 velocity=0.0

Commit message: snakes

File: body.urdf (robot description, URDF)
Before this commit: robot robot, 5 links, 4 joints
Links:
- added link link10, mass 1; collision box size=0.8427964447325348 0.6893618411453469 0.3357726378936953; visual box size=0.8427964447325348 0.6893618411453469 0.3357726378936953
- added link link5, mass 1; collision box size=0.7935544140214699 0.9078156599856063 0.38450472364261784; visual box size=0.7935544140214699 0.9078156599856063 0.38450472364261784
- added link link6, mass 1; collision box size=0.22879892273802338 0.7569405505160435 0.03627416365085151; visual box size=0.22879892273802338 0.7569405505160435 0.03627416365085151
- added link link7, mass 1; collision box size=0.0746318899278543 0.6733761538311768 0.2679273066037763; visual box size=0.0746318899278543 0.6733761538311768 0.2679273066037763
- added link link8, mass 1; collision box size=0.7053755599325728 0.6927977199310974 0.15293445291548635; visual box size=0.7053755599325728 0.6927977199310974 0.15293445291548635
- added link link9, mass 1; collision box size=0.9379777064039747 0.47878385553666325 0.18126342926678285; visual box size=0.9379777064039747 0.47878385553666325 0.18126342926678285
- link link0: geometry collision box size=0.9368688720538945 0.4985460401410696 0.46140115615055216; visual box size=0.9368688720538945 0.4985460401410696 0.46140115615055216
- link link1: geometry collision box size=0.38091511896625174 0.5319232145167948 0.09742158252837263; visual box size=0.38091511896625174 0.5319232145167948 0.09742158252837263
- link link2: geometry collision box size=0.03595903457108196 0.396830604656638 0.41460453521399804; visual box size=0.03595903457108196 0.396830604656638 0.41460453521399804
- link link3: geometry collision box size=0.44263671808579785 0.27220554659076757 0.10402974565926781; visual box size=0.44263671808579785 0.27220554659076757 0.10402974565926781
- link link4: geometry collision box size=0.977204759213608 0.9437375958840766 0.29117196214498653; visual box size=0.977204759213608 0.9437375958840766 0.29117196214498653
Joints:
- added joint link4_link5: type revolute, parent link4, child link5, origin xyz=-0.977204759213608 -0.20847067629804833 -0.24920794831794746 rpy=0 0 0, axis 0 0 1, limit lower=-3.14159 upper=3.14159 effort=0.0 velocity=0.0
- added joint link5_link6: type revolute, parent link5, child link6, origin xyz=-0.7935544140214699 0.12601229464749766 0.21833585012443052 rpy=0 0 0, axis 0 0 1, limit lower=-3.14159 upper=3.14159 effort=0.0 velocity=0.0
- added joint link6_link7: type revolute, parent link6, child link7, origin xyz=-0.22879892273802338 -0.08154850784059339 0.017726369404282842 rpy=0 0 0, axis 0 0 1, limit lower=-3.14159 upper=3.14159 effort=0.0 velocity=0.0
- added joint link7_link8: type revolute, parent link7, child link8, origin xyz=-0.0746318899278543 -0.042403407750486566 0.045234771406931495 rpy=0 0 0, axis 0 0 1, limit lower=-3.14159 upper=3.14159 effort=0.0 velocity=0.0
- added joint link8_link9: type revolute, parent link8, child link9, origin xyz=-0.7053755599325728 -0.1965335079616513 0.004078475742013719 rpy=0 0 0, axis 0 0 1, limit lower=-3.14159 upper=3.14159 effort=0.0 velocity=0.0
- added joint link9_link10: type revolute, parent link9, child link10, origin xyz=-0.9379777064039747 0.20480268419219264 -0.03891467673078475 rpy=0 0 0, axis 0 0 1, limit lower=-3.14159 upper=3.14159 effort=0.0 velocity=0.0
- joint link0_link1: origin xyz=-0.02429744666783773 0 1 rpy=0 0 0 -> xyz=-0.46843443602694723 -0.014571833283286982 0.895551382296907 rpy=0 0 0
- joint link1_link2: origin xyz=-0.4325252736494065 0 0 rpy=0 0 0 -> xyz=-0.38091511896625174 -0.3089352976541222 0.015836245159624285 rpy=0 0 0
- joint link2_link3: origin xyz=-0.137498004971097 0 0 rpy=0 0 0 -> xyz=-0.03595903457108196 0.13217706210425068 0.030599182385357734 rpy=0 0 0
- joint link3_link4: origin xyz=-0.9921424383479781 0 0 rpy=0 0 0 -> xyz=-0.44263671808579785 0.07035387135754051 -0.0014530211520287738 rpy=0 0 0

Commit message: final_project biped

File: body.urdf (robot description, URDF)
Before this commit: robot robot, 9 links, 8 joints
Links:
- removed link BackLeg
- removed link BackLowerLeg
- removed link FrontLeg
- removed link FrontLowerLeg
- removed link LeftLowerLeg
- removed link RightLowerLeg
- added link LeftArm, mass 1; collision box size=0.5 0.25 0.25; visual box size=0.5 0.25 0.25
- added link LowerLeft, mass 1; collision box size=0.25 0.25 0.5; visual box size=0.25 0.25 0.5
- added link LowerRight, mass 1; collision box size=0.25 0.25 0.5; visual box size=0.25 0.25 0.5
- added link RightArm, mass 1; collision box size=0.5 0.25 0.25; visual box size=0.5 0.25 0.25
- link LeftLeg: geometry collision box size=0.25 0.25 0.5; visual box size=0.25 0.25 0.5
- link RightLeg: geometry collision box size=0.25 0.25 0.5; visual box size=0.25 0.25 0.5
- link Torso: geometry collision box size=0.5 0.5 1; visual box size=0.5 0.5 1
Joints:
- removed joint BackLeg_BackLowerLeg
- removed joint FrontLeg_FrontLowerLeg
- removed joint LeftLeg_LeftLowerLeg
- removed joint RightLeg_RightLowerLeg
- removed joint Torso_BackLeg
- removed joint Torso_FrontLeg
- added joint LeftLeg_LowerLeft: type revolute, parent LeftLeg, child LowerLeft, origin xyz=0 0 -0.5 rpy=0 0 0, axis 1 0 0, limit lower=-3.14159 upper=3.14159 effort=0.0 velocity=0.0
- added joint RightLeg_LowerRight: type revolute, parent RightLeg, child LowerRight, origin xyz=0 0 0 rpy=0 0 0, axis 1 0 0, limit lower=-3.14159 upper=3.14159 effort=0.0 velocity=0.0
- added joint Torso_LeftArm: type revolute, parent Torso, child LeftArm, origin xyz=-0.25 0 2 rpy=0 0 0, axis 0 1 0, limit lower=-3.14159 upper=3.14159 effort=0.0 velocity=0.0
- added joint Torso_RightArm: type revolute, parent Torso, child RightArm, origin xyz=0.25 0 2 rpy=0 0 0, axis 0 1 0, limit lower=-3.14159 upper=3.14159 effort=0.0 velocity=0.0
- joint Torso_LeftLeg: axis 0 1 0 -> 1 0 0; origin xyz=-0.5 0 1 rpy=0 0 0 -> xyz=-0.25 0 1.5 rpy=0 0 0
- joint Torso_RightLeg: axis 0 1 0 -> 1 0 0; origin xyz=0.5 0 1 rpy=0 0 0 -> xyz=0.25 0 1 rpy=0 0 0
